File: optical-keyboard-mx.kicad_pcb (KiCad board)
At the start: 2 copper layers, 9.5 x 10 mm, 388 parts, among them M1 LED, M10 LED, M11 LED, M12 LED, M13 LED, M14 LED, M15 LED, M16 LED, M17 LED, M18 LED, M19 LED, M2 LED, M20 LED, M21 LED, M22 LED, M23 LED, M24 LED, M25 LED, M26 LED, M27 LED, M28 LED, M29 LED, M3 LED, M30 LED, M31 LED, M32 LED, M33 LED, M34 LED, M35 LED, M36 LED, M37 LED, M38 LED, M39 LED, M4 LED, M40 LED, M41 LED, M42 LED, M43 LED, M44 LED, M45 LED, M46 LED, M47 LED, M48 LED, M49 LED, M5 LED, M50 LED, M51 LED, M52 LED, M53 LED, M54 LED, M55 LED, M56 LED, M57 LED, M58 LED, M59 LED, M6 LED, M60 LED, M61 LED, M62 LED, M63 LED, M64 LED, M65 LED, M66 LED, M67 LED, M68 LED, M69 LED, M7 LED, M70 LED, M71 LED, M72 LED, M73 LED, M74 LED, M8 LED, M9 LED, Q1 Q_Photo_NPN, Q10 Q_Photo_NPN, Q11 Q_Photo_NPN, Q12 Q_Photo_NPN, Q13 Q_Photo_NPN, Q14 Q_Photo_NPN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

Commit message: Added traces through python script
D  MyFootprints.pretty/Gateron_Sw_1.25u.kicad_mod
D  MyFootprints.pretty/Gateron_Sw_1.5u.kicad_mod
D  MyFootprints.pretty/Gateron_Sw_1.75u.kicad_mod
M  MyFootprints.pretty/Gateron_Sw_1u.kicad_mod
D  MyFootprints.pretty/Gateron_Switch_Basic.kicad_mod
M  optical-keyboard-mx.kicad_pcb
M  optical-keyboard-mx.kicad_prl
M  placemx.py
Parts:
- moved U1 47.8 mm to (-6.00, 56.0), turned to 0 degrees
- moved M44 7.89 mm to (285.0, 32.9)
- moved Q44 7.89 mm to (288.4, 38.0)
- moved RL44 7.89 mm to (293.3, 41.5)
- moved S44 7.89 mm to (285.0, 38.0)
- moved D44 7.89 mm to (281.6, 38.0)
- moved Q43 3.08 mm to (267.0, 38.0)
- moved D43 3.08 mm to (260.2, 38.0)
- moved M43 3.08 mm to (263.6, 32.9)
- moved RL43 3.08 mm to (271.9, 41.5)
- moved S43 3.08 mm to (263.6, 38.0)
- moved D74 0.80 mm to (291.1, 76.0)
- moved RL74 0.80 mm to (302.8, 79.5)
- moved S74 0.80 mm to (294.5, 76.0)
- moved M74 0.80 mm to (294.5, 70.9)
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Routing:
- net (no net): track 434.4 -> 0.00 mm
- net CA4: track 76.8 -> 269.0 mm
- net CA3: track 64.8 -> 255.3 mm
- net GND: track 0.00 -> 177.6 mm, vias 0 -> 148
- net CB8: track 25.6 -> 74.3 mm, vias 2 -> 4
- net CB3: track 180.8 -> 228.3 mm, vias 2 -> 4
- net CB7: track 116.5 -> 160.4 mm, vias 6 -> 8
- net CB6: track 114.1 -> 155.7 mm, vias 6 -> 8
- net CB2: track 205.4 -> 233.2 mm, vias 4 -> 6
- net CB1: track 238.0 -> 265.8 mm, vias 4 -> 6
- net /row3: track 380.0 -> 356.1 mm
- net CB5: track 272.5 -> 255.9 mm
- net CB4: track 215.5 -> 225.8 mm
- net /col15: track 120.8 -> 115.1 mm
- net /col14: track 160.5 -> 164.9 mm
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Other:
- board size 9.5 x 10 mm -> 10 x 9.5 mm

Commit message: Python scripts to add curved tracks
Script to place mouting holes, draw edge cuts.

A  MyFootprints.pretty/SMTSO_M1.6.kicad_mod
A  MyFootprints.pretty/SMTSO_M2.kicad_mod
A  drawborder.py
M  optical-keyboard-mx.kicad_pcb
M  optical-keyboard-mx.kicad_prl
M  optical-keyboard-mx.kicad_sch
A  placeholes.py
M  placemx.py
Parts:
- added H1: MountingHole, MyFootprints:SMTSO_M2, F.Cu at (147.5, 48.0)
- added H10: MountingHole, MyFootprints:SMTSO_M2, F.Cu at (303.8, 85.8)
- added H11: MountingHole, MyFootprints:SMTSO_M2, F.Cu at (199.5, -9.00)
- added H12: MountingHole, MyFootprints:SMTSO_M2, F.Cu at (71.2, 48.0)
- added H13: MountingHole, MyFootprints:SMTSO_M2, F.Cu at (247.0, 85.5)
- added H14: MountingHole, MyFootprints:SMTSO_M2, F.Cu at (42.8, 85.5)
- added H15: MountingHole, MyFootprints:SMTSO_M2, F.Cu at (104.5, -9.00)
- added H16: MountingHole, MyFootprints:SMTSO_M2, F.Cu at (247.2, 9.75)
- added H17: MountingHole, MyFootprints:SMTSO_M2, F.Cu at (57.0, 10.0)
- added H18: MountingHole, MyFootprints:SMTSO_M2, F.Cu at (152.2, 10.2)
- added H2: MountingHole, MyFootprints:SMTSO_M2, F.Cu at (173.2, 86.5)
- added H3: MountingHole, MyFootprints:SMTSO_M2, F.Cu at (223.5, 48.0)
- added H4: MountingHole, MyFootprints:SMTSO_M2, F.Cu at (299.8, 41.5)
- added H5: MountingHole, MyFootprints:SMTSO_M2, F.Cu at (101.8, 86.5)
- added H6: MountingHole, MyFootprints:SMTSO_M2, F.Cu at (-11.8, 85.2)
- added H7: MountingHole, MyFootprints:SMTSO_M2, F.Cu at (8.00, 22.2)
- added H8: MountingHole, MyFootprints:SMTSO_M2, F.Cu at (9.50, -9.00)
- added H9: MountingHole, MyFootprints:SMTSO_M2, F.Cu at (294.5, -9.00)
- moved U1 2.25 mm to (-6.00, 53.8)
Routing:
- net /row3: track 356.1 -> 372.1 mm
- net CB5: track 255.9 -> 271.9 mm
- net CB4: track 225.8 -> 241.8 mm
- net CB3: track 228.3 -> 244.3 mm
- net CB2: track 233.2 -> 249.2 mm
- net CB1: track 265.8 -> 281.8 mm

Commit message: Add python script to draw edge cuts
M  MyFootprints.pretty/BlackPill_STLINK_Down.kicad_mod
A  MyFootprints.pretty/MountingHole_1.7mm_M1.6_Pad.kicad_mod
A  MyFootprints.pretty/MountingHole_2.2mm_M2_ISO7380_Pad.kicad_mod
A  MyFootprints.pretty/PinHeader_1x04_P2.54mm_Vertical.kicad_mod
A  MyFootprints.pretty/PinHeader_1x08_P2.54mm_Vertical.kicad_mod
M  MySymbols.kicad_sym
M  drawborder.py
A  mounting-hw.kicad_sch
M  optical-keyboard-mx.kicad_pcb
M  optical-keyboard-mx.kicad_prl
M  optical-keyboard-mx.kicad_pro
M  optical-keyboard-mx.kicad_sch
M  placeholes.py
Parts:
- removed H18: MountingHole, MyFootprints:SMTSO_M2
- added HS1: MountingHoleStdoffM2, MyFootprints:MountingHole_2.2mm_M2_ISO7380_Pad, F.Cu at (331.4, 80.2)
- added HS2: MountingHoleStdoffM2, MyFootprints:MountingHole_2.2mm_M2_ISO7380_Pad, F.Cu at (346.5, 85.2)
- added HS3: MountingHoleStdoffM2, MyFootprints:MountingHole_2.2mm_M2_ISO7380_Pad, F.Cu at (336.4, 85.2)
- added HS4: MountingHoleStdoffM2, MyFootprints:MountingHole_2.2mm_M2_ISO7380_Pad, F.Cu at (341.5, 80.2)
- added HS5: MountingHoleStdoffM2, MyFootprints:MountingHole_2.2mm_M2_ISO7380_Pad, F.Cu at (336.4, 80.2)
- added HS6: MountingHoleStdoffM2, MyFootprints:MountingHole_2.2mm_M2_ISO7380_Pad, F.Cu at (331.4, 85.2)
- added HS7: MountingHoleStdoffM2, MyFootprints:MountingHole_2.2mm_M2_ISO7380_Pad, F.Cu at (346.5, 80.2)
- added HS8: MountingHoleStdoffM2, MyFootprints:MountingHole_2.2mm_M2_ISO7380_Pad, F.Cu at (341.5, 85.2)
- added J1: Conn_01x04, MyFootprints:PinHeader_1x04_P2.54mm_Vertical, F.Cu at (320.7, 114.6)
- added J2: Conn_01x08, MyFootprints:PinHeader_1x08_P2.54mm_Vertical, F.Cu at (320.8, 76.7)
- moved H17 258.3 mm to (304.0, 85.5)
- moved H13 252.7 mm to (-5.70, 85.5)
- moved H7 239.3 mm to (247.0, 10.0)
- moved H12 232.8 mm to (304.0, 48.0)
- moved H9 230.4 mm to (71.2, 48.0)
- moved H6 180.2 mm to (152.0, 10.0)
- moved H10 161.0 mm to (147.2, 48.0)
- moved H1 149.5 mm to (9.50, -9.50)
- moved H2 118.1 mm to (104.5, -9.50)
- moved H15 100.2 mm to (137.8, 85.5)
- moved H5 88.6 mm to (57.0, 10.0)
- moved H16 78.2 mm to (228.0, 85.5)
- moved H3 62.3 mm to (199.5, -9.50)
- moved H11 61.7 mm to (223.2, 48.0)
- moved H4 51.3 mm to (294.5, -9.50)
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Routing:
- net /row1: track 367.4 -> 288.3 mm
- net /row4: track 376.9 -> 297.8 mm
- net /row3: track 372.1 -> 293.0 mm
- net /row2: track 350.7 -> 277.2 mm
- net CB1: track 281.8 -> 216.8 mm
- net CB5: track 271.9 -> 209.8 mm
- net CA4: track 269.0 -> 209.7 mm
- net /row5: track 264.8 -> 208.3 mm
- net CB2: track 249.2 -> 195.6 mm
- net CB3: track 244.3 -> 190.6 mm
- net CB4: track 241.8 -> 188.1 mm
- net CA3: track 255.3 -> 201.6 mm
- net CA2: track 260.1 -> 206.4 mm
- net CA5: track 220.8 -> 170.0 mm
- net CA1: track 240.9 -> 192.9 mm
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Other:
- board size 10 x 9.5 mm -> 324.8 x 186 mm

Commit message: More scripts to draw border and place footprint
M  drawborder.py
M  mounting-hw.kicad_sch
M  optical-keyboard-mx.kicad_pcb
M  optical-keyboard-mx.kicad_sch
M  placefp.py
 D placefpg.mx
M  placeholes.py
Parts:
- added J10: Conn_01x04, MyFootprints:PinHeader_1x04_P2.54mm_Vertical, F.Cu at (235.0, 87.5)
- added J11: Conn_01x04, MyFootprints:PinHeader_1x04_P2.54mm_Vertical, F.Cu at (289.4, 87.5)
- added J12: Conn_01x04, MyFootprints:PinHeader_1x04_P2.54mm_Vertical, F.Cu at (-4.25, 169.0)
- added J13: Conn_01x04, MyFootprints:PinHeader_1x04_P2.54mm_Vertical, F.Cu at (53.6, 169.0)
- added J14: Conn_01x04, MyFootprints:PinHeader_1x04_P2.54mm_Vertical, F.Cu at (214.2, 169.0)
- added J15: Conn_01x04, MyFootprints:PinHeader_1x04_P2.54mm_Vertical, F.Cu at (272.1, 169.0)
- added J16: Conn_01x04, MyFootprints:PinHeader_1x04_P2.54mm_Vertical, F.Cu at (-4.25, 117.0)
- added J17: Conn_01x04, MyFootprints:PinHeader_1x04_P2.54mm_Vertical, F.Cu at (53.6, 117.0)
- added J18: Conn_01x04, MyFootprints:PinHeader_1x04_P2.54mm_Vertical, F.Cu at (214.2, 117.0)
- added J19: Conn_01x04, MyFootprints:PinHeader_1x04_P2.54mm_Vertical, F.Cu at (272.1, 117.0)
- added J20: Conn_01x04, MyFootprints:PinHeader_1x04_P2.54mm_Vertical, F.Cu at (-13.2, 137.1)
- added J21: Conn_01x04, MyFootprints:PinHeader_1x04_P2.54mm_Vertical, F.Cu at (70.2, 137.1)
- added J22: Conn_01x04, MyFootprints:PinHeader_1x04_P2.54mm_Vertical, F.Cu at (205.2, 137.1)
- added J23: Conn_01x04, MyFootprints:PinHeader_1x04_P2.54mm_Vertical, F.Cu at (288.8, 137.1)
- added J24: Conn_01x04, MyFootprints:PinHeader_1x04_P2.54mm_Vertical, F.Cu at (7.50, 5.12)
- added J25: Conn_01x04, MyFootprints:PinHeader_1x04_P2.54mm_Vertical, F.Cu at (296.5, 5.12)
- added J26: Conn_01x04, MyFootprints:PinHeader_1x04_P2.54mm_Vertical, F.Cu at (61.5, 28.5)
- added J27: Conn_01x04, MyFootprints:PinHeader_1x04_P2.54mm_Vertical, F.Cu at (137.5, 28.5)
- added J28: Conn_01x04, MyFootprints:PinHeader_1x04_P2.54mm_Vertical, F.Cu at (232.5, 28.5)
- added J29: Conn_01x04, MyFootprints:PinHeader_1x04_P2.54mm_Vertical, F.Cu at (105.3, 101.9)
- added J3: Conn_01x04, MyFootprints:PinHeader_1x04_P2.54mm_Vertical, F.Cu at (111.5, -11.5)
- added J30: Conn_01x04, MyFootprints:PinHeader_1x04_P2.54mm_Vertical, F.Cu at (162.7, 104.7)
- added J4: Conn_01x04, MyFootprints:PinHeader_1x04_P2.54mm_Vertical, F.Cu at (184.9, -11.5)
- added J5: Conn_01x04, MyFootprints:PinHeader_1x04_P2.54mm_Vertical, F.Cu at (206.5, -11.5)
- added J6: Conn_01x04, MyFootprints:PinHeader_1x04_P2.54mm_Vertical, F.Cu at (279.9, -11.5)
- added J7: Conn_01x04, MyFootprints:PinHeader_1x04_P2.54mm_Vertical, F.Cu at (9.13, 87.5)
- added J8: Conn_01x04, MyFootprints:PinHeader_1x04_P2.54mm_Vertical, F.Cu at (68.8, 87.5)
- added J9: Conn_01x04, MyFootprints:PinHeader_1x04_P2.54mm_Vertical, F.Cu at (213.4, 87.5)
- J2: value Conn_01x08 -> Conn_01x04; footprint MyFootprints:PinHeader_1x08_P2.54mm_Vertical -> MyFootprints:PinHeader_1x04_P2.54mm_Vertical
- moved HS1 355.9 mm to (-13.2, 169.0)
- moved HS5 351.6 mm to (-13.2, 117.0)
- moved J1 329.3 mm to (16.5, -11.5), turned to 90 degrees
- moved HS2 288.7 mm to (70.2, 169.0)
- moved HS6 263.0 mm to (70.2, 117.0)
- moved J2 247.2 mm to (89.9, -11.5), turned to 90 degrees
- moved HS3 155.7 mm to (205.2, 169.0)
- moved HS7 146.0 mm to (205.2, 117.0)
- moved HS4 103.3 mm to (288.8, 169.0)
- moved HS8 61.6 mm to (288.8, 117.0)
- moved R1 49.0 mm to (121.0, 71.0)
- moved C1 38.5 mm to (112.0, 76.0), turned to 90 degrees
- moved C2 38.5 mm to (118.0, 76.0), turned to 90 degrees
- moved H13 29.4 mm to (23.8, 85.5)
- moved H14 19.0 mm to (61.8, 85.5)
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Routing:
- net CB5: track 209.8 -> 305.2 mm, vias 6 -> 12
- net CB1: track 216.8 -> 127.1 mm, vias 6 -> 0
- net /row5: track 208.3 -> 214.5 mm, vias 0 -> 1
- net /col5: track 121.6 -> 125.6 mm
- net CA5: track 170.0 -> 173.4 mm
- net CA6: track 77.5 -> 80.1 mm
- net GND: track 177.6 -> 176.4 mm, vias 148 -> 147
- net /col9: track 119.2 -> 120.2 mm
Other:
- outline, holes or cut-outs redrawn

Commit message: Tracks laid, wrist support and switch plate
M  MyFootprints.pretty/BlackPill_STLINK_Down.kicad_mod
M  MyFootprints.pretty/SMTSO_M1.6.kicad_mod
M  MyFootprints.pretty/SMTSO_M2.kicad_mod
M  MyFootprints.pretty/Switch_Cutout.kicad_mod
D  MyFootprints.pretty/Switch_Cutout_1.25u.kicad_mod
D  MyFootprints.pretty/Switch_Cutout_1.5u.kicad_mod
D  MyFootprints.pretty/Switch_Cutout_1.75u.kicad_mod
M  MySymbols.kicad_sym
M  drawborder.py
M  led_driver.kicad_sch
M  mounting-hw.kicad_sch
M  optical-keyboard-mx.kicad_pcb
M  optical-keyboard-mx.kicad_prl
M  optical-keyboard-mx.kicad_pro
M  optical-keyboard-mx.kicad_sch
M  placefp.py
 D placefpg.mx
M  placeholes.py
A  switch-plate/.gitignore
A  switch-plate/fp-lib-table
A  switch-plate/switch-plate.kicad_pcb
A  switch-plate/switch-plate.kicad_prl
A  switch-plate/switch-plate.kicad_pro
A  switch-plate/switch-plate.kicad_sch
A  switch-plate/sym-lib-table
M  switch.kicad_sch
A  wrist-support/.gitignore
A  wrist-support/fp-lib-table
A  wrist-support/sym-lib-table
A  wrist-support/wrist-support.kicad_pcb
A  wrist-support/wrist-support.kicad_prl
A  wrist-support/wrist-support.kicad_pro
A  wrist-support/wrist-support.kicad_sch
Parts:
- removed J1, J10, J11, J12, J13, J14, J15, J16, J17, J18, J19, J2, J20, J21, J22, J23, J24, J25, J26, J27, J28, J29, J3, J30, J4, J5, J6, J7, J8, J9: Conn_01x04, MyFootprints:PinHeader_1x04_P2.54mm_Vertical
- H1, H10, H11, H12, H13, H14, H15, H16, H17, H2, H3, H4, H5, H6, H7, H8, H9: value MountingHole -> MountingHoleStdoffM2
- HS1, HS2, HS3, HS4, HS5, HS6, HS7, HS8: value MountingHoleStdoffM2 -> MountingHoleSprt; footprint MyFootprints:MountingHole_2.2mm_M2_ISO7380_Pad -> MyFootprints:SMTSO_M2
- moved HS4 225.0 mm to (69.8, 117.5)
- moved HS5 225.0 mm to (205.8, 168.5)
- moved HS3 224.0 mm to (-12.8, 117.5)
- moved HS6 224.0 mm to (288.2, 168.5)
- moved R1 26.8 mm to (147.4, 75.3), turned to 45 degrees
- moved R2 17.3 mm to (156.3, 65.2), turned to 180 degrees
- moved R3 13.9 mm to (156.2, 67.6)
- moved R5 10.1 mm to (145.5, 73.5), turned to -45 degrees
- moved R4 9.99 mm to (159.1, 68.0), turned to -90 degrees
- moved C4 7.08 mm to (164.1, 67.9)
- moved R6 7.04 mm to (151.0, 79.5), turned to -135 degrees
- moved C2 5.62 mm to (123.0, 73.4), turned to 180 degrees
- moved C3 1.16 mm to (149.7, 77.9), turned to 45 degrees
- moved H15 1.00 mm to (137.8, 86.5)
- moved HS1 0.71 mm to (-12.8, 168.5)
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Connections:
- U1 pad 39: GND1 -> GND
Routing:
- net /col15: track 92.5 -> 413.7 mm, vias 4 -> 5
- net /col14: track 125.4 -> 420.2 mm, vias 5 -> 7
- net VCC: track 0.00 -> 282.4 mm, vias 0 -> 7
- net /col13: track 120.5 -> 395.8 mm, vias 5 -> 6
- net /col12: track 119.2 -> 375.6 mm, vias 5 -> 6
- net /col11: track 119.2 -> 370.5 mm, vias 5 -> 8
- net /col8: track 94.4 -> 337.5 mm, vias 4 -> 6
- net /col10: track 119.2 -> 349.1 mm, vias 5 -> 8
- net /col9: track 120.2 -> 320.2 mm, vias 5 -> 9
- net /col6: track 94.4 -> 293.1 mm, vias 4 -> 6
- net /col7: track 115.9 -> 314.2 mm, vias 5 -> 6
- net /row1: track 288.3 -> 477.7 mm, vias 0 -> 1
- net CB8: track 54.6 -> 241.4 mm, vias 4 -> 5
- net GND: track 176.4 -> 357.3 mm, vias 147 -> 154
- net CA1: track 192.9 -> 362.9 mm, vias 4 -> 8
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- added copper zone on B.Cu, net GND
Other:
- outline, holes or cut-outs redrawn
