File: wrist-support/wrist-support.kicad_sch (KiCad schematic)
At the start: 4 parts

Commit message: Add gerbers and assembly files
M  .gitignore
M  MyFootprints.pretty/MountingHole_2.2mm_M2_ISO7380_Pad.kicad_mod
M  MySymbols.kicad_sym
M  README.md
M  drawborder.py
A  jlcpcb/gerber/optical-keyboard-mx-B_Cu.gbl
A  jlcpcb/gerber/optical-keyboard-mx-B_Mask.gbs
A  jlcpcb/gerber/optical-keyboard-mx-B_Paste.gbp
A  jlcpcb/gerber/optical-keyboard-mx-B_Silkscreen.gbo
A  jlcpcb/gerber/optical-keyboard-mx-Edge_Cuts.gm1
A  jlcpcb/gerber/optical-keyboard-mx-F_Cu.gtl
A  jlcpcb/gerber/optical-keyboard-mx-F_Mask.gts
A  jlcpcb/gerber/optical-keyboard-mx-F_Paste.gtp
A  jlcpcb/gerber/optical-keyboard-mx-F_Silkscreen.gto
A  jlcpcb/gerber/optical-keyboard-mx-NPTH-drl_map.gbr
A  jlcpcb/gerber/optical-keyboard-mx-NPTH.drl
A  jlcpcb/gerber/optical-keyboard-mx-PTH-drl_map.gbr
A  jlcpcb/gerber/optical-keyboard-mx-PTH.drl
M  led_driver.kicad_sch
M  mounting-hw.kicad_sch
M  optical-keyboard-mx.kicad_pcb
M  optical-keyboard-mx.kicad_sch
M  placefp.py
M  switch-plate/.gitignore
A  switch-plate/jlcpcb/gerber/switch-plate-B_Cu.gbl
A  switch-plate/jlcpcb/gerber/switch-plate-B_Mask.gbs
A  switch-plate/jlcpcb/gerber/switch-plate-B_Paste.gbp
A  switch-plate/jlcpcb/gerber/switch-plate-B_Silkscreen.gbo
A  switch-plate/jlcpcb/gerber/switch-plate-Edge_Cuts.gm1
A  switch-plate/jlcpcb/gerber/switch-plate-F_Cu.gtl
A  switch-plate/jlcpcb/gerber/switch-plate-F_Mask.gts
A  switch-plate/jlcpcb/gerber/switch-plate-F_Paste.gtp
A  switch-plate/jlcpcb/gerber/switch-plate-F_Silkscreen.gto
A  switch-plate/jlcpcb/gerber/switch-plate-NPTH-drl_map.gbr
A  switch-plate/jlcpcb/gerber/switch-plate-NPTH.drl
A  switch-plate/jlcpcb/gerber/switch-plate-PTH-drl_map.gbr
A  switch-plate/jlcpcb/gerber/switch-plate-PTH.drl
M  switch-plate/switch-plate.kicad_pcb
M  switch-plate/switch-plate.kicad_prl
M  switch.kicad_sch
M  wrist-support/.gitignore
A  wrist-support/jlcpcb/gerber/wrist-support-B_Cu.gbl
A  wrist-support/jlcpcb/gerber/wrist-support-B_Mask.gbs
A  wrist-support/jlcpcb/gerber/wrist-support-B_Paste.gbp
A  wrist-support/jlcpc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
Parts:
- HS1, HS2, HS3, HS4: footprint MyFootprints:MountingHole_2.2mm_M2_jlcpcb -> MyFootprints:MountingHole_2.2mm_M2_ISO7380_Pad
Changed lines of the file:
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@@
       (effects (font (size 1.27 1.27)) (justify left))
     )
-    (property "Footprint" "MyFootprints:MountingHole_2.2mm_M2_jlcpcb" (id 2) (at 86.36 67.31 0)
+    (property "Footprint" "MyFootprints:MountingHole_2.2mm_M2_ISO7380_Pad" (id 2) (at 86.36 67.31 0)
       (effects (font (size 1.27 1.27)) hide)
     )
@@
       (effects (font (size 1.27 1.27)) (justify left))
     )
-    (property "Footprint" "MyFootprints:MountingHole_2.2mm_M2_jlcpcb" (id 2) (at 97.79 67.31 0)
+    (property "Footprint" "MyFootprints:MountingHole_2.2mm_M2_ISO7380_Pad" (id 2) (at 97.79 67.31 0)
       (effects (font (size 1.27 1.27)) hide)
     )
@@
       (effects (font (size 1.27 1.27)) (justify left))
     )
-    (property "Footprint" "MyFootprints:MountingHole_2.2mm_M2_jlcpcb" (id 2) (at 74.93 67.31 0)
+    (property "Footprint" "MyFootprints:MountingHole_2.2mm_M2_ISO7380_Pad" (id 2) (at 74.93 67.31 0)
       (effects (font (size 1.27 1.27)) hide)
     )
@@
       (effects (font (size 1.27 1.27)) (justify left))
     )
-    (property "Footprint" "MyFootprints:MountingHole_2.2mm_M2_jlcpcb" (id 2) (at 63.5 67.31 0)
+    (property "Footprint" "MyFootprints:MountingHole_2.2mm_M2_ISO7380_Pad" (id 2) (at 63.5 67.31 0)
       (effects (font (size 1.27 1.27)) hide)
     )
@@
   (symbol_instances
     (path "/de802840-e6bf-4733-8fb7-6ceb379d06d2"
-      (reference "HS1") (unit 1) (value "MountingHoleSprt") (footprint "MyFootprints:MountingHole_2.2mm_M2_jlcpcb")
+      (reference "HS1") (unit 1) (value "MountingHoleSprt") (footprint "MyFootprints:MountingHole_2.2mm_M2_ISO7380_Pad")
     )
     (path "/7b389730-92d7-4079-9df3-df7004eb26b8"
-      (reference "HS2") (unit 1) (value "MountingHoleSprt") (footprint "MyFootprints:MountingHole_2.2mm_M2_jlcpcb")
+      (reference "HS2") (unit 1) (value "MountingHoleSprt") (footprint "MyFootprints:MountingHole_2.2mm_M2_ISO7380_Pad")
     )
     (path "/69976d14-2978-4dda-85dc-df37583aa900"
-      (reference "HS3") (unit 1) (value "MountingHoleSprt") (footprint "MyFootprints:MountingHole_2.2mm_M2_jlcpcb")
+      (reference "HS3") (unit 1) (value "MountingHoleSprt") (footprint "MyFootprints:MountingHole_2.2mm_M2_ISO7380_Pad")
     )
     (path "/718cd874-b021-4fb3-960d-ba4bffb2786f"
-      (reference "HS4") (unit 1) (value "MountingHoleSprt") (footprint "MyFootprints:MountingHole_2.2mm_M2_jlcpcb")
+      (reference "HS4") (unit 1) (value "MountingHoleSprt") (footprint "MyFootprints:MountingHole_2.2mm_M2_ISO7380_Pad")
     )
   )
